Commit message: add modification

File: rotors_description/urdf/multirotor_base_REAL.xacro (robot description, xacro)
@@ -47,5 +47,5 @@
       </inertial>
       <visual>
-        <origin xyz="0 0 -0.06995" rpy="0 0 0" />
+        <origin xyz="0 0 0" rpy="0 0 0" />
         <geometry>
           <xacro:if value="${use_mesh_file}">
@@ -53,5 +53,5 @@
           </xacro:if>
           <xacro:unless value="${use_mesh_file}">
-            <box size="${body_width} ${0.147.5} ${0.13991}"/> <!-- [m] [m] [m] -->
+            <box size="${body_width} ${body_width} ${body_height}"/> <!-- [m] [m] [m] -->
           </xacro:unless>
         </geometry>
@@ -60,5 +60,5 @@
         <origin xyz="0 0 0" rpy="0 0 0" />
         <geometry>
-          <box size="${body_width} ${0.08} ${0.13991}" /> <!-- [m] [m] [m] -->
+          <box size="${body_width} ${body_width} ${body_height}" /> <!-- [m] [m] [m] -->
         </geometry>
       </collision>
